File: Charger/Charger.kicad_pcb (KiCad board)
At the start: 2 copper layers, 115.1 x 70.3 mm, 30 parts, among them J1 IN, J2 OUT, Q1 2N3904, Q2 IRFZ44N, Q3 2N3906, U1 TL494

Commit message: Add files via upload
Parts:
- added R12: 100, Resistors_THT:R_Axial_DIN0207_L6.3mm_D2.5mm_P7.62mm_Horizontal, F.Cu at (97.0, 66.7)
Connections:
- Q1 pad 3: Net-(C1-Pad1) -> Net-(Q1-Pad3)
Routing:
- net Net-(C1-Pad1): track 24.7 -> 12.0 mm
- net Net-(Q1-Pad3): track 0.00 -> 6.54 mm
- net VCC: track 87.5 -> 89.8 mm
Changed lines of the file:
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@@
 (kicad_pcb (version 4) (host pcbnew 4.0.6)
   (general
-    (links 57)
+    (links 58)
     (no_connects 0)
-    (area 72.949999 36.23794 189.4994 111.962001)
+    (area 72.949999 41.530199 188.162001 111.962001)
     (thickness 1.6)
     (drawings 9)
-    (tracks 130)
+    (tracks 132)
     (zones 0)
-    (modules 30)
-    (nets 19)
+    (modules 31)
+    (nets 20)
   )
   (page A4)
@@
   (net 17 "Net-(R8-Pad2)")
   (net 18 IFB)
+  (net 19 "Net-(Q1-Pad3)")
   (net_class Default "This is the default net class."
     (clearance 0.2)
@@
     (add_net "Net-(D2-Pad1)")
     (add_net "Net-(Q1-Pad1)")
+    (add_net "Net-(Q1-Pad3)")
     (add_net "Net-(R2-Pad1)")
     (add_net "Net-(R7-Pad2)")
@@
       (net 10 SIG))
     (pad 3 thru_hole oval (at 2.54 0 270) (size 0.9 1.5) (drill 0.6) (layers *.Cu *.Mask)
-      (net 1 "Net-(C1-Pad1)"))
+      (net 19 "Net-(Q1-Pad3)"))
     (pad 1 thru_hole rect (at 0 0 270) (size 0.9 1.5) (drill 0.6) (layers *.Cu *.Mask)
       (net 11 "Net-(Q1-Pad1)"))
@@
     (fp_line (start -0.508 -2.54) (end 0 -2.54) (layer F.Cu) (width 0.381))
   )
+  (module Resistors_THT:R_Axial_DIN0207_L6.3mm_D2.5mm_P7.62mm_Horizontal (layer F.Cu)
+    (at 97.0026 66.675 270)
+    (descr "Resistor, Axial_DIN0207 series, Axial, Horizontal, pin pitch=7.62mm, 0.25W = 1/4W, length*diameter=6.3*2.5mm^2, http://cdn-reichelt.de/documents/datenblatt/B400/1_4W%23YAG.pdf")
+    (tags "Resistor Axial_DIN0207 series Axial Horizontal pin pitch 7.62mm 0.25W = 1/4W length 6.3mm diameter 2.5mm")
+    (fp_text reference R12 (at 3.81 -2.31 270) (layer F.SilkS)
+      (effects (font (size 1 1) (thickness 0.15)))
+    )
+    (fp_text value 100 (at 3.81 2.31 270) (layer F.Fab)
+      (effects (font (size 1 1) (thickness 0.15)))
+    )
+    (fp_line (start 0.66 -1.25) (end 0.66 1.25) (layer F.Fab) (width 0.1))
+    (fp_line (start 0.66 1.25) (end 6.96 1.25) (layer F.Fab) (width 0.1))
+    (fp_line (start 6.96 1.25) (end 6.96 -1.25) (layer F.Fab) (width 0.1))
+    (fp_line (start 6.96 -1.25) (end 0.66 -1.25) (layer F.Fab) (width 0.1))
+    (fp_line (start 0 0) (end 0.66 0) (layer F.Fab) (width 0.1))
+    (fp_line (start 7.62 0) (end 6.96 0) (layer F.Fab) (width 0.1))
+    (fp_line (start 0.6 -0.98) (end 0.6 -1.31) (layer F.SilkS) (width 0.12))
+    (fp_line (start 0.6 -1.31) (end 7.02 -1.31) (layer F.SilkS) (width 0.12))
+    (fp_line (start 7.02 -1.31) (end 7.02 -0.98) (layer F.SilkS) (width 0.12))
+    (fp_line (start 0.6 0.98) (end 0.6 1.31) (layer F.SilkS) (width 0.12))
+    (fp_line (start 0.6 1.31) (end 7.02 1.31) (layer F.SilkS) (width 0.12))
+    (fp_line (start 7.02 1.31) (end 7.02 0.98) (layer F.SilkS) (width 0.12))
+    (fp_line (start -1.05 -1.6) (end -1.05 1.6) (layer F.CrtYd) (width 0.05))
+    (fp_line (start -1.05 1.6) (end 8.7 1.6) (layer F.CrtYd) (width 0.05))
+    (fp_line (start 8.7 1.6) (end 8.7 -1.6) (layer F.CrtYd) (width 0.05))
+    (fp_line (start 8.7 -1.6) (end -1.05 -1.6) (layer F.CrtYd) (width 0.05))
+    (pad 1 thru_hole circle (at 0 0 270) (size 1.6 1.6) (drill 0.8) (layers *.Cu *.Mask)
+      (net 19 "Net-(Q1-Pad3)"))
+    (pad 2 thru_hole oval (at 7.62 0 270) (size 1.6 1.6) (drill 0.8) (layers *.Cu *.Mask)
+      (net 1 "Net-(C1-Pad1)"))
+    (model ${KISYS3DMOD}/Resistors_THT.3dshapes/R_Axial_DIN0207_L6.3mm_D2.5mm_P7.62mm_Horizontal.wrl
+      (at (xyz 0 0 0))
+      (scale (xyz 0.393701 0.393701 0.393701))
+      (rotate (xyz 0 0 0))
+    )
+  )
   (gr_text "7.8V TO 39V\n0-5A " (at 97.3582 104.5464) (layer F.SilkS)
     (effects (font (size 1.5 1.5) (thickness 0.3)))
@@
   (gr_line (start 188.087 41.656) (end 188.087 111.887) (angle 90) (layer Edge.Cuts) (width 0.15))
   (gr_line (start 73.279 41.656) (end 188.087 41.656) (angle 90) (layer Edge.Cuts) (width 0.15))
-  (segment (start 90.8812 77.6732) (end 94.4626 77.6732) (width 0.25) (layer F.Cu) (net 1))
-  (segment (start 100.2538 66.6496) (end 103.5304 66.6496) (width 0.25) (layer F.Cu) (net 1))
-  (segment (start 99.2378 67.6656) (end 100.2538 66.6496) (width 0.25) (layer F.Cu) (net 1))
-  (segment (start 99.2378 72.898) (end 99.2378 67.6656) (width 0.25) (layer F.Cu) (net 1))
-  (segment (start 94.4626 77.6732) (end 99.2378 72.898) (width 0.25) (layer F.Cu) (net 1))
+  (segment (start 90.8812 77.6732) (end 93.6244 77.6732) (width 0.25) (layer B.Cu) (net 1) (status 400000))
+  (segment (start 93.6244 77.6732) (end 97.0026 74.295) (width 0.25) (layer B.Cu) (net 1) (status 800000))
   (segment (start 86.5124 77.4446) (end 90.6526 77.4446) (width 0.25) (layer B.Cu) (net 1))
   (segment (start 90.6526 77.4446) (end 90.8812 77.6732) (width 0.25) (layer B.Cu) (net 1))
-  (segment (start 90.8812 67.5132) (end 91.5162 67.5132) (width 0.25) (layer B.Cu) (net 3) (status C00000))
-  (segment (start 91.5162 67.5132) (end 95.4024 63.627) (width 0.25) (layer B.Cu) (net 3) (status 400000))
-  (segment (start 95.4024 63.627) (end 95.4024 60.4266) (width 0.25) (layer B.Cu) (net 3))
+  (segment (start 107.5944 80.8736) (end 102.997 80.8736) (width 0.25) (layer B.Cu) (net 3) (status 400000))
+  (segment (start 95.4024 68.707) (end 95.4024 63.0174) (width 0.25) (layer B.Cu) (net 3))
+  (segment (start 96.8756 70.1802) (end 95.4024 68.707) (width 0.25) (layer B.Cu) (net 3))
+  (segment (start 98.425 70.1802) (end 96.8756 70.1802) (width 0.25) (layer B.Cu) (net 3))
+  (segment (start 99.9236 71.6788) (end 98.425 70.1802) (width 0.25) (layer B.Cu) (net 3))
+  (segment (start 99.9236 77.8002) (end 99.9236 71.6788) (width 0.25) (layer B.Cu) (net 3))
+  (segment (start 102.997 80.8736) (end 99.9236 77.8002) (width 0.25) (layer B.Cu) (net 3))
+  (segment (start 90.8812 67.5132) (end 91.5162 67.5132) (width 0.25) (layer B.Cu) (net 3))
+  (segment (start 91.5162 67.5132) (end 95.4024 63.627) (width 0.25) (layer B.Cu) (net 3))
+  (segment (start 95.4024 63.627) (end 95.4024 63.0174) (width 0.25) (layer B.Cu) (net 3))
+  (segment (start 95.4024 63.0174) (end 95.4024 60.4266) (width 0.25) (layer B.Cu) (net 3))
   (segment (start 92.964 60.4266) (end 95.4024 60.4266) (width 1.2) (layer B.Cu) (net 3))
   (segment (start 95.4024 60.4266) (end 97.1042 60.4266) (width 1.2) (layer B.Cu) (net 3))
@@
   (segment (start 84.3534 60.4266) (end 82.5754 58.6486) (width 1.2) (layer B.Cu) (net 3))
   (segment (start 90.8812 67.5132) (end 90.8812 67.3354) (width 0.25) (layer B.Cu) (net 3))
-  (segment (start 83.4898 59.7408) (end 82.5754 58.6486) (width 0.25) (layer B.Cu) (net 3) (status 800000))
-  (segment (start 107.5944 80.8736) (end 103.5558 80.8736) (width 0.25) (layer B.Cu) (net 3))
-  (segment (start 93.5736 67.5132) (end 90.8812 67.5132) (width 0.25) (layer B.Cu) (net 3))
-  (segment (start 94.9706 68.9102) (end 93.5736 67.5132) (width 0.25) (layer B.Cu) (net 3))
-  (segment (start 94.9706 72.2884) (end 94.9706 68.9102) (width 0.25) (layer B.Cu) (net 3))
-  (segment (start 103.5558 80.8736) (end 94.9706 72.2884) (width 0.25) (layer B.Cu) (net 3))
+  (segment (start 83.4898 59.7408) (end 82.5754 58.6486) (width 0.25) (layer B.Cu) (net 3))
   (segment (start 123.0376 88.265) (end 114.9858 88.265) (width 0.25) (layer B.Cu) (net 3))
   (segment (start 114.9858 88.265) (end 107.5944 80.8736) (width 0.25) (layer B.Cu) (net 3))
@@
   (segment (start 155.4226 105.8672) (end 131.9022 105.8672) (width 0.25) (layer F.Cu) (net 18))
   (segment (start 167.386 93.9038) (end 155.4226 105.8672) (width 0.25) (layer F.Cu) (net 18))
+  (segment (start 97.0026 66.675) (end 103.505 66.675) (width 0.25) (layer B.Cu) (net 19) (status C00000))
+  (segment (start 103.505 66.675) (end 103.5304 66.6496) (width 0.25) (layer B.Cu) (net 19) (status C00000))
   (zone (net 2) (net_name GND) (layer F.Cu) (hatch edge 0.508)
     (connect_pads (clearance 0.508))
